File: MoistureMeasure/moistureMeasure.brd (EAGLE design)
At the start: 49.5 x 32.4 mm, 8 parts, among them IC1 74HC14D, Q1 BC847BSMD

Commit message: mainBoard update
Parts:
- moved C1 16.1 mm to (12.1, 11.7)
- moved C2 16.1 mm to (9.84, 12.7)
- moved D1 16.1 mm to (3.17, 24.4)
- moved Q1 16.1 mm to (6.99, 29.5)
- moved R1 16.1 mm to (3.49, 29.5)
- moved R3 16.1 mm to (6.03, 19.1)
- moved IC1 16.1 mm to (8.89, 19.4)
- moved R2 16.1 mm to (8.26, 25.1)

Commit message: moisture and main board updates
Routing:
- net C1: track 12.2 -> 15.6 mm
- net N$1: track 2.93 -> 0.00 mm
- net C2: track 12.3 -> 13.0 mm
- net GND: track 25.3 -> 24.9 mm, vias 1 -> 0
- net 5VDC: track 21.2 -> 20.8 mm, vias 0 -> 1
Other:
- outline, holes or cut-outs redrawn
- board text added: "GND"
- board text added: "MoistureMeasure v1.1"
- board text added: "SEN"
- board text added: "UB"
- board text added: "WaterCtrl"
- board text added: "github.com/janhieber/WaterCtrl"
