File: MainBoard/mainBoard.sch (EAGLE design)
At the start: 21 parts, among them IC2 LM317

Commit message: mainBoard updates
Parts:
- removed C2: 100n, rcl:C-EU050-024X044
- added C10: 1u, rcl:C-EUC0805
- added C6, C7: 22p, rcl:C-EUC0805
- added C8: 100n, rcl:C-EUC0805
- added Q1: 8MHz, crystal:CRYSTALHC49UP
- added SV1: ESP8266, con-lstb:MA04-2
- added X1: PWR12, con-ptr500:AK500/2
- C1, C11: value 470u/25V -> 47u/25V
- C3, C4, C5: device rcl:C-EU050-024X044 -> rcl:C-EUC0603K
- C9: device rcl:C-EU050-024X044 -> rcl:C-EUC0805
- R1, R3, R7: device rcl:R-EU_R0805W -> rcl:R-EU_R0805
Connections:
- new net OSC_IN: C6.1, Q1.1, U$1.PF0/OSC_IN
- new net OSC_OUT: C7.1, Q1.2, U$1.PF1/OSC_OUT
- net +12V: now also X1-1.KL
- net +3V3: now also C10.1, C8.1, U$1.VDDA, U$1.VDD_1, U$1.VDD_2; no longer C2.1
- net GND: now also C10.2, C6.2, C7.2, C8.2, U$1.BOOT0, U$1.VSSA, U$1.VSS_1, U$1.VSS_2, X1-2.KL; no longer C2.2

Commit message: some more main board updates
Parts:
- added C12, C13, C14, C15, C16: 100n, rcl:C-EUC0805
- added Q10, Q2, Q4, Q6, Q8: BC547, transistor-npn:BC547
- added Q11, Q3, Q5, Q7, Q9: (no value), transistor-power:P-MOSFET-SO8
- added R10, R14, R18, R22, R4: 18k, rcl:R-EU_R0805
- added R11, R15, R19, R23, R6: 1k2, rcl:R-EU_R0805
- added R12, R16, R20, R24, R8: 560, rcl:R-EU_R0805
- added R13, R17, R2, R21, R9: 10k, rcl:R-EU_R0805
- added X2, X3, X4, X5, X6: MSTBA2, con-phoenix-508:MSTBA2
Connections:
- new net N$10: Q6.C, R16.1
- new net N$11: Q6.B, R13.2, R14.2
- new net N$13: C15.2, Q9.G, R19.1, R20.2
- new net N$14: Q8.C, R20.1
- new net N$15: Q8.B, R17.2, R18.2
- new net N$16: C16.2, Q11.G, R23.1, R24.2
- new net N$17: Q10.C, R24.1
- new net N$18: Q10.B, R21.2, R22.2
- new net N$2: C13.2, Q5.G, R11.1, R12.2
- new net N$3: C12.2, Q3.G, R6.1, R8.2
- new net N$4: Q2.C, R8.1
- new net N$5: Q2.B, R2.2, R4.2
- new net N$6: Q4.C, R12.1
- new net N$7: Q4.B, R10.2, R9.2
- new net N$8: C14.2, Q7.G, R15.1, R16.2
- new net PA15: SV1.8
- new net PA4: R13.1, U$1.PA4
- new net PA5: R17.1, U$1.PA5
- new net PA6: R21.1, U$1.PA6
- new net PF4: R2.1, U$1.PF4
- new net PF5: R9.1, U$1.PF5
- new net WP1: Q3.D, X2-1.1
- new net WP2: Q5.D, X3-1.1
- new net WP3: Q7.D, X4-1.1
- new net WP4: Q9.D, X5-1.1
- new net WP5: Q11.D, X6-1.1
- net +12V: now also C12.1, C13.1, C14.1, C15.1, C16.1, Q11.S, Q3.S, Q5.S, Q7.S, Q9.S, R11.2, R15.2, R19.2, R23.2, R6.2
- net +3V3: now also SV1.2
- net GND: now also Q10.E, Q2.E, Q4.E, Q6.E, Q8.E, R10.1, R14.1, R18.1, R22.1, R4.1, SV1.7, X2-2.1, X3-2.1, X4-2.1, X5-2.1, X6-2.1
- net PA14: now also SV1.1

Commit message: mainBoard update
Parts:
- added IC1: 74HC151D, 74xx-eu:74HC151D
- added IC3: 74HC138D, 74xx-eu:74HC138D
- added J1, J2, J3, J4, J5, J6, J7, J8: 22-05-7038-03, con-molex:22-05-7038-03
- added R25: 18k, rcl:R-EU_R0805
Connections:
- new net FREQ: IC1A.Y
- new net S1_3V: IC3A.Y0, J1-1.S
- new net S1_DAT: IC1A.D0, J1-2.S
- new net S2_3V: IC3A.Y1, J2-1.S
- new net S2_DAT: IC1A.D1, J2-2.S
- new net S3_3V: IC3A.Y2, J3-1.S
- new net S3_DAT: IC1A.D2, J3-2.S
- new net S4_3V: IC3A.Y3, J4-1.S
- new net S4_DAT: IC1A.D3, J4-2.S
- new net S5_3V: IC3A.Y4, J5-1.S
- new net S5_DAT: IC1A.D4, J5-2.S
- new net S6_3V: IC3A.Y5, J6-1.S
- new net S6_DAT: IC1A.D5, J6-2.S
- new net S7_3V: IC3A.Y6, J7-1.S
- new net S7_DAT: IC1A.D6, J7-2.S
- new net S8_3V: IC3A.Y7, J8-1.S
- new net S8_DAT: IC1A.D7, J8-2.S
- new net SEN_ENABLE: IC3A.G1, R25.2
- new net SEN_SEL0: IC1A.A, IC3A.A
- new net SEN_SEL1: IC1A.B, IC3A.B
- new net SEN_SEL2: IC1A.C, IC3A.C
- net +3V3: now also IC1P.VCC, IC3P.VCC
- net GND: now also IC1A.G, IC1P.GND, IC3A.G2A, IC3A.G2B, IC3P.GND, J1-3.S, J2-3.S, J3-3.S, J4-3.S, J5-3.S, J6-3.S, J7-3.S, J8-3.S, R25.1

Commit message: mainboard updates
Parts:
- added C2: 22p, rcl:C-EUC0805
Changed lines of the file:
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@@
 <part name="GND33" library="supply1" deviceset="GND" device=""/>
 <part name="GND29" library="supply1" deviceset="GND" device=""/>
+<part name="C2" library="rcl" deviceset="C-EU" device="C0805" value="22p">
+<attribute name="R" value="SPR-0805 240"/>
+</part>
 </parts>
 <sheets>
@@
 <instance part="GND1" gate="1" x="124.46" y="35.56"/>
 <instance part="+3V1" gate="G$1" x="86.36" y="33.02"/>
+<instance part="C2" gate="G$1" x="35.56" y="101.6">
+<attribute name="R" x="35.56" y="101.6" size="1.778" layer="96" display="off"/>
+</instance>
 </instances>
 <busses>

Commit message: mainboard updates
Parts:
- removed C2: 22p, rcl:C-EUC0805
- added C17: 100n, rcl:C-EUC0805
- added Q12: BC847ASMD, transistor-npn:BC847ASMD
- added Q13: (no value), transistor-power:P-MOSFET-SO8
- added R26: 10k, rcl:R-EU_R0805
- added R27: 18k, rcl:R-EU_R0805
- added R28: 1k2, rcl:R-EU_R0805
- added R29: 560, rcl:R-EU_R0805
- added X7: MSTBA2, con-phoenix-508:MSTBA2
- Q10, Q2, Q4, Q6, Q8: value BC547 -> BC847ASMD; device transistor-npn:BC547 -> transistor-npn:BC847ASMD
Connections:
- new net N$19: C17.2, Q13.G, R28.1, R29.2
- new net N$21: Q12.C, R29.1
- new net N$22: Q12.B, R26.2, R27.2
- new net PA7: R26.1
- new net WP6: Q13.D, X7-1.1
- net +12V: now also C17.1, Q13.S, R28.2
- net GND: now also Q12.E, R27.1, X7-2.1
Other:
- moved on the sheet: C12, C13, C14, C15, C16, Q10, Q11, Q2, Q3, Q4, Q5, Q6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

Commit message: mainboard updates
Parts:
- added R30, R31: 2R4 1/4W, rcl:R-EU_R1206
- added R32, R33, R34, R35: 18k, rcl:R-EU_R0805
- added S1, S2, S3, S4: (no value), switch-omron:10-XX
- added SV2: DISP_A, con-lstb:MA03-1
- added SV3: DISP_B, con-lstb:MA03-1
- added SV4: DISP_C, con-lstb:MA04-1
- added SV5: DISP_D, con-lstb:MA07-1
- IC3: value 74HC138D -> 74HC238
Connections:
- new net D_ENABLE: SV5.4
- new net D_IM1: SV4.3
- new net D_IM2: SV4.4
- new net D_RESET: SV5.1
- new net D_RS: SV5.2
- new net D_RW: SV5.3
- new net D_SCLK_SCL: SV5.5
- new net D_SID_SDAIN: SV5.6
- new net D_SOD_SDAOUT: SV5.7
- new net N$23: R30.1, R31.1, SV2.1, SV2.2, SV2.3
- new net SW1: R32.2, S1.P, S1.P1
- new net SW2: R33.2, S2.P, S2.P1
- new net SW3: R34.2, S3.P, S3.P1
- new net SW4: R35.2, S4.P, S4.P1
- net +3V3: now also IC3A.G1, R25.2, R30.2, R31.2, S1.S, S1.S1, S2.S, S3.S, S4.S, SV4.2; no longer JP3.1
- net GND: now also R32.1, R33.1, R34.1, R35.1, SV3.1, SV3.2, SV3.3, SV4.1; no longer IC1A.G, IC3A.G2A, IC3A.G2B, R25.1
- net PA7: now also U$1.PA7
- net SEN_ENABLE: now also IC1A.G, IC3A.G2A, IC3A.G2B, R25.1; no longer IC3A.G1, R25.2
Other:
- note added: "Output not inverting. Wrong symbol"
- moved on the sheet: C3, C4, C5, C6, C7, JP1, JP2, JP3, Q1, R25, SV1, U$1

Commit message: mainboard updates
Parts:
- added D1, D2, D3, D4, D5, D6: (no value), diode:SCHOTTKY-DIODESMD
- added J10, J11, J12, J13, J14, J15, J16, J9: 22-05-7038-03, con-molex:22-05-7038-03
- added R36: 18k, rcl:R-EU_R0805
- added X10, X11, X12, X13, X8, X9: MSTBA2, con-phoenix-508:MSTBA2
- JP1: device pinhead:PINHD-1X5 -> pinhead:PINHD-1X6
- R1: value 47 -> 100
Connections:
- net PA13 renamed SWDIO
- net RX1 renamed USART1_RX
- net TX1 renamed USART1_TX
- removed net PA14: JP1.2, SV1.1, U$1.SWCLK/PA14
- removed net PA15: SV1.8
- removed net PA9: U$1.PA9
- new net N$24: U$1.PA11
- new net N$25: U$1.PA12
- new net SWCLK: JP1.2, U$1.SWCLK/PA14
- new net USART2_RX: SV1.8, U$1.PA3
- new net USART2_TX: SV1.1, U$1.PA2
- new net WIFI_RESET: R36.2, SV1.4, SV1.6, U$1.PA1
- net FREQ: now also U$1.PA9
- net GND: now also D1.A, D2.A, D3.A, D4.A, D5.A, D6.A, J10-3.S, J11-3.S, J12-3.S, J13-3.S, J14-3.S, J15-3.S, J16-3.S, J9-3.S, R36.1, X10-2.1, X11-2.1, X12-2.1, X13-2.1, X8-2.1, X9-2.1
- net S1_3V: now also J9-1.S
- net S1_DAT: now also J9-2.S
- net S2_3V: now also J10-1.S
- net S2_DAT: now also J10-2.S
- net S3_3V: now also J11-1.S
- net S3_DAT: now also J11-2.S
- net S4_3V: now also J12-1.S
- net S4_DAT: now also J12-2.S
- net S5_3V: now also J13-1.S
- net S5_DAT: now also J13-2.S
- net S6_3V: now also J14-1.S
- net S6_DAT: now also J14-2.S
- net S7_3V: now also J15-1.S
- net S7_DAT: now also J15-2.S
- net S8_3V: now also J16-1.S
- net S8_DAT: now also J16-2.S
- net SEN_ENABLE: now also U$1.PB15
- net SEN_SEL0: now also U$1.PB14
- net SEN_SEL1: now also U$1.PB13
- net SEN_SEL2: now also U$1.PB12
- net WP1: now also D1.C, X8-1.1
- net WP2: now also D2.C, X9-1.1
- net WP3: now also D3.C, X10-1.1
- net WP4: now also D4.C, X11-1.1
- net WP5: now also D5.C, X12-1.1
- net WP6: now also D6.C, X13-1.1
Other:
- moved on the sheet: C12, C13, C14, C15, C16, C17, J1-1, J1-2, J1-3, J2-1, J2-2, J2-3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

Commit message: mainboard updates...
Parts:
- C1, C11: R (none) -> VF 47/25 P-D
- C10: R (none) -> X7R-G0805 1,0/25
- C12, C13, C14, C15, C16, C17, C8, C9: R (none) -> X7R-G0805 100N
- C3, C4, C5: R (none) -> X7R-G0603 100N
- C6, C7: R (none) -> NPO-G0805 22P
- D1, D2, D3, D4, D5, D6: R (none) -> B 340 F
- IC1: R (none) -> SMD HC 151
- IC2: R (none) -> LM317EMP
- IC3: R (none) -> SMD HC 238
- J1, J2, J3, J4, J5, J6, J7, J8: R (none) -> PSS 254/3W
- JP1: R (none) -> MPE 087-1-006
- JP2: R (none) -> MPE 087-1-002
- JP3: R (none) -> MPE 087-1-004
- LED1: R (none) -> SMD-LED 0805 GN
- Q1: R (none) -> 8,0000-HC49-SMD
- Q10, Q12, Q2, Q4, Q6, Q8: R (none) -> BC 547A
- Q11, Q13, Q3, Q5, Q7, Q9: R (none) -> IRF 9332
- R1: R (none) -> SMD-0805 100
- R10, R14, R18, R22, R25, R27, R32, R33, R34, R35, R36, R4: R (none) -> SMD-0805 18,0K
- R11, R15, R19, R23, R28, R6: R (none) -> SMD-0805 1,20K
- R12, R16, R20, R24, R29, R8: R (none) -> SMD-0805 560
- R13, R17, R2, R21, R26, R9: R (none) -> SMD-0805 10,0K
- R3: R (none) -> SPR-0805 300
- R30, R31: R (none) -> SMD 1/4W 2,4
- R5: R (none) -> 64Y-200
- R7: R (none) -> SPR-0805 240
- S1, S2, S3, S4: R (none) -> TASTER 9302
- SV1: R (none) -> MPE 094-2-008
- SV2: R (none) -> BL 1X20G7 2,54
- U$1: value STM32F051 -> STM32 F051 R4T6
- X1: R (none) -> AKL 101-02
- X2, X3, X4, X5, X6, X7: R (none) -> AKL 230-02
Other:
- note added: "Stecker: Reichelt 8x PSK 254/3W"
