File: MainBoard/mainBoard.brd (EAGLE design)
At the start: 149.6 x 99.3 mm, 87 parts, among them IC2 74HC238, IC3 74HC151D, J1 22-05-7038-03, J2 22-05-7038-03, J3 22-05-7038-03, J4 22-05-7038-03, J5 22-05-7038-03, J6 22-05-7038-03, J7 22-05-7038-03, J8 22-05-7038-03, Q1 BC847ASMD, Q10 BC847ASMD, Q2 BC847ASMD, Q5 BC847ASMD, Q6 BC847ASMD, Q9 BC847ASMD, X1 PWR12, X2 MSTBA2, X3 MSTBA2, X4 MSTBA2, X5 MSTBA2, X6 MSTBA2, X7 MSTBA2

Commit message: board updates
Parts:
- added JP2: UART_STM, pinhead:1X03
- JP1: value (none) -> UART_RPI; device pinhead:1X04 -> pinhead:1X03
- moved JP1 84.8 mm to (76.5, 81.5), turned to 90 degrees
- moved Q1 48.9 mm to (25.1, 13.2)
- moved R7 45.4 mm to (31.2, 13.5), turned to 180 degrees
- moved R5 45.2 mm to (22.4, 12.2), turned to 90 degrees
- moved R9 44.8 mm to (28.2, 13.2), turned to 270 degrees
- moved X2 43.5 mm to (36.3, 5.08)
- moved R11 42.7 mm to (26.4, 10.2), turned to 180 degrees
- moved C7 41.5 mm to (22.4, 8.13)
- moved Q3 41.0 mm to (26.7, 5.08), turned to 0 degrees
- moved D2 35.6 mm to (37.3, 4.32)
- moved D7 25.4 mm to (107.4, -16.0)
- moved D3 25.4 mm to (84.1, -16.0)
- moved D4 25.4 mm to (55.4, -16.0)
- moved D5 25.4 mm to (95.8, -16.0)
- moved D6 25.4 mm to (67.1, -16.0)
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Connections:
- removed net 5V: U$2.3
- removed net ERROR_LED: LED2.A
- removed net N$23: PCB1.1
- new net LED_ERR: LED2.A, U$2.4
- new net N$30: PCB1.39
- new net SPI1_MISO: PCB1.21, U$2.30
- new net SPI1_MOSI: PCB1.19, U$2.29
- new net SPI1_SCK: PCB1.23, U$2.31
- new net STM_RXD: JP2.2, U$2.14
- new net STM_TXD: JP2.1, U$2.15
- net +5V: now also U$2.3; no longer JP1.1
- net 3V3: no longer PCB1.17
- net GND: now also JP1.3, JP2.3; no longer JP1.4, PCB1.39
- net RPI_RXD: now also JP1.2; no longer JP1.3
- net RPI_TXD: now also JP1.1; no longer JP1.2
Routing:
- net +15V: track 96.0 -> 214.3 mm
- net +5V: track 70.0 -> 126.5 mm, vias 1 -> 3
- net STM_RXD: track 0.00 -> 54.0 mm, vias 0 -> 1
- net RPI_TXD: track 0.00 -> 53.0 mm, vias 0 -> 1
- net STM_TXD: track 0.00 -> 48.5 mm, vias 0 -> 1
- net 3V3: track 0.00 -> 48.0 mm, vias 0 -> 2
- net LED_ERR: track 0.00 -> 34.0 mm, vias 0 -> 1
- net RPI_RXD: track 20.1 -> 53.6 mm, vias 0 -> 1
- net SPI1_SCK: track 0.00 -> 25.1 mm
- net SPI1_MOSI: track 0.00 -> 18.6 mm
- net SPI1_MISO: track 0.00 -> 11.7 mm
- net WP1: track 6.38 -> 15.9 mm
- net N$3: track 13.3 -> 16.4 mm, vias 0 -> 2
- net N$9: track 0.00 -> 2.32 mm
- net GND: track 1.95 -> 0.00 mm, vias 9 -> 59
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- removed copper zone on layer 1, net WP1
Other:
- outline, holes or cut-outs redrawn
- board text added: "TX RX GND"
- board text removed: "5V TX RX GND"
- board text removed: "rPi UART"

Commit message: mainboard updates
Parts:
- added IC1: 74HC238, 74xx-eu:SO16
- R3: value 100 -> 150
- moved H2 50.5 mm to (93.7, 93.7)
- moved Q1 46.0 mm to (71.1, 13.2)
- moved Q3 46.0 mm to (72.6, 5.08)
- moved R11 46.0 mm to (72.4, 10.2)
- moved R9 46.0 mm to (74.2, 13.2)
- moved X2 46.0 mm to (82.3, 5.08)
- moved D2 46.0 mm to (83.3, 4.32)
- moved C7 46.0 mm to (68.3, 8.13)
- moved R5 46.0 mm to (68.3, 12.2)
- moved R7 46.0 mm to (77.2, 13.5)
- moved R4 43.0 mm to (82.0, 47.8), turned to 90 degrees
- moved IC2 42.8 mm to (83.8, 56.1)
- moved IC3 42.6 mm to (83.6, 68.3)
- moved J1 41.7 mm to (94.2, 85.9)
- moved J2 41.7 mm to (94.2, 77.7)
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Connections:
- net SEN_SEL0 renamed SEN_A0
- net SEN_SEL1 renamed SEN_A1
- net SEN_SEL2 renamed SEN_A2
- removed net +3V3: R4.2
- removed net PA4: R7.1
- removed net PA6: R15.1
- removed net PA7: R23.1
- removed net PA8: R24.1
- removed net PB0: R8.1
- removed net PB10: R16.1
- new net N$24: IC2.4, IC2.5
- new net PWM: IC1.6, U$2.35
- new net PWM_A0: IC1.1, U$2.38
- new net PWM_A1: IC1.2, U$2.37
- new net PWM_A2: IC1.3, U$2.36
- new net RPI_NRST: PCB1.P$1, U$2.39
- new net VCC: IC1.16
- new net WP1C: IC1.15, R7.1
- new net WP2C: IC1.14, R15.1
- new net WP3C: IC1.13, R23.1
- new net WP4C: IC1.11, R8.1
- new net WP5C: IC1.12, R16.1
- new net WP6C: IC1.10, R24.1
- net +5V: no longer IC2.6
- net GND: now also IC1.4, IC1.5, IC1.8, IC3.7, PCB1.P$2, PCB1.PE_BL, PCB1.PE_BR, PCB1.PE_TR, R4.1
- net SEN_ENABLE: now also IC2.6, R4.2; no longer IC2.4, IC2.5, IC3.7, R4.1
Routing:
- net +15V: track 214.3 -> 173.4 mm
- net PWM_A1: track 0.00 -> 39.9 mm
- net PWM_A0: track 0.00 -> 38.5 mm
- net PWM_A2: track 0.00 -> 35.2 mm
- net PWM: track 0.00 -> 34.9 mm
- net RPI_NRST: track 0.00 -> 9.94 mm
- net +5V: track 126.5 -> 127.0 mm
Other:
- board size 149.6 x 99.3 mm -> 99.3 x 99.3 mm
