File: MainBoard/20150430_bak/mainBoard.sch (EAGLE design)
At the start: 103 parts, among them IC2 74HC238, IC3 74HC151D, J1 22-05-7038-03, J2 22-05-7038-03, J3 22-05-7038-03, J4 22-05-7038-03, J5 22-05-7038-03, J6 22-05-7038-03, J7 22-05-7038-03, J8 22-05-7038-03, Q1 BC847ASMD, Q10 BC847ASMD, Q2 BC847ASMD, Q5 BC847ASMD, Q6 BC847ASMD, Q9 BC847ASMD, U1 STM32F0DISCOVERY, X1 PWR12, X2 MSTBA2, X3 MSTBA2, X4 MSTBA2, X5 MSTBA2, X6 MSTBA2, X7 MSTBA2

Commit message: mainboard redesign
Parts:
- removed D7: (no value), diode:SCHOTTKY-DIODESMC
- removed KK1: SK104-PAD, heatsink:SK104-PAD
- removed PCB1: RASPBERRY_PI_B+_TPLACE, RASPBERRY_PI_Bplus:RASPBERRY_PI_B+_TPLACE
- removed U$2: PSK 254/3W, extra:DUMMY_BOM
- removed U1: STM32F0DISCOVERY, extra:STM32F0DISCOVERY
- added C13, C14, C15, C16, C17: 100n, rcl:C-EUC0805
- added C18: 4.7u/35V, rcl:CPOL-EUB
- added C19: 10n, rcl:C-EUC0603K
- added C2, C20: 100n, rcl:C-EUC0603K
- added IC1: 74HC151D, 74xx-eu:74HC151D
- added IC4: FT232RL, ftdichip:FT232RL
- added J10, J11, J12, J13, J14, J15, J16, J9: 22-05-7038-03, con-molex:22-05-7038-03
- added JP2: EXTPWR, pinhead:PINHD-1X2
- added JP3: UART, pinhead:PINHD-1X4
- added Q13: (no value), transistor-power:P-MOSFET-SO8
- added R30, R31: 2R4 1/4W, rcl:R-EU_R1206
- added R32, R33, R34, R35, R36: 18k, rcl:R-EU_R0805
- added R37, R38: EMI 60Ohm Ferrit, rcl:R-EU_R0603
- added R39: 100, rcl:R-EU_R0805
- added S1, S2, S3, S4: (no value), switch-omron:10-XX
- added SJ1: (no value), jumper:SJ
- added SV1: ESP8266, con-lstb:MA04-2
- added SV2: DISP_A, con-lstb:MA03-1
- added SV3: DISP_B, con-lstb:MA03-1
- added SV4: DISP_C, con-lstb:MA04-1
- added SV5: DISP_D, con-lstb:MA07-1
- added U$18, U$19: Kontakte (20Stk), extra:DUMMY_BOM
- added X10, X11, X12, X13, X8, X9: MSTBA2, con-phoenix-508:MSTBA2
- added X15: MINI-USB-SCHIELD-32005-301, con-cypressindustries:MINI-USB-SCHIELD-32005-301
- C10: value 100n -> 1u; R X7R-G0805 100N -> X7R-G0805 1,0/25
- C11: value 100n -> 47u/25V; device rcl:C-EUC0805 -> rcl:CPOL-EUD; R X7R-G0805 100N -> VF 47/25 P-D
- C3: value 47u/25V -> 100n; device rcl:CPOL-EUD -> rcl:C-EUC0603K; R VF 47/25 P-D -> X7R-G0603 100N
- C4, C5: device rcl:C-EUC0805 -> rcl:C-EUC0603K; R X7R-G0805 100N -> X7R-G0603 100N
- C6: value 1u -> 22p; R X7R-G0805 1,0/25 -> NPO-G0805 22P
- C7: value 100n -> 22p; R X7R-G0805 100N -> NPO-G0805 22P
- D1: device diode:DIODE-MELF-MLL41 -> diode:SCHOTTKY-DIODESMC; R 1N 4002 SMD -> B 340 F
- IC2: value 74HC238 -> LM317; device 74xx-eu:74HC138D -> v-reg:LM317MBSTT3; R SMD HC 238 -> LM317EMP
- IC3: value 74HC151D -> 74HC238; device 74xx-eu:74HC151D -> 74xx-eu:74HC138D; R SMD HC 151 -> SMD HC 238
- JP1: value (none) -> SWD; device pinhead:PINHD-1X4 -> pinhead:PINHD-1X6; R (none) -> MPE 087-1-006
- Q1: value BC847ASMD -> 8MHz; device transistor-npn:BC847ASMD -> crystal:CRYSTALHC49UP; R BC 847A SMD -> 8,0000-HC49-SMD
- Q12, Q4, Q8: value (none) -> BC847ASMD; device transistor-power:P-MOSFET-SO8 -> transistor-npn:BC847ASMD; R IRF 9332 -> BC 847A SMD
- Q5, Q9: value BC847ASMD -> (none); device transistor-npn:BC847ASMD -> transistor-power:P-MOSFET-SO8; R BC 847A SMD -> IRF 9332
- R1: value 750 -> 100; R SPR-0805 750 -> SMD-0805 100
- R11, R19, R28: value 560 -> 1k2; R SMD-0805 560 -> SMD-0805 1,20K
- R13, R21: value 1k2 -> 10k; R SMD-0805 1,20K -> SMD-0805 10,0K
- R14, R22: value 1k2 -> 18k; R SMD-0805 1,20K -> SMD-0805 18,0K
- R15, R23: value 10k -> 1k2; R SMD-0805 10,0K -> SMD-0805 1,20K
- R16, R24, R8: value 10k -> 560; R SMD-0805 10,0K -> SMD-0805 560
- R17, R26, R9: value 18k -> 10k; R SMD-0805 18,0K -> SMD-0805 10,0K
- R2: value 240 -> 10k; R SPR-0805 240 -> SMD-0805 10,0K
- R27: value 560 -> 18k; R SMD-0805 560 -> SMD-0805 18,0K
- R29: value 100 -> 560; R SMD-0805 100 -> SMD-0805 560
- R3: value 100 -> 300; R SMD-0805 100 -> SPR-0805 300
- R5: value 1k2 -> 200; device rcl:R-EU_R0805 -> pot:TRIM_EU-S64Y; R SMD-0805 1,20K -> 64Y-200
- R7: value 10k -> 240; R SMD-0805 10,0K -> SPR-0805 240
- U$1: value LM350 -> STM32 F051 R4T6; device extra:LM350 -> stm32F:STM32F051; R LM 350-220 -> (none)
- U$10: value Kontakte (20Stk) -> PSK 254/3W; R PSK-KONTAKTE -> PSK 254/3W
- U$11: value Kontakte (20Stk) -> EA DOGM204W-A; R PSK-KONTAKTE -> EA DOGM204W-A
- U$3: BOM (none) -> yes
Connections:
- removed net +15V: C1.+, C10.1, C11.1, C12.1, C3.+, C4.1, C7.1, C8.1, C9.1, D1.C, Q11.S, Q12.S, Q3.S, Q4.S, Q7.S, Q8.S, R13.2, R14.2, R21.2, R22.2, R5.2, R6.2, U$1.IN, X1-1.KL
- removed net +5V: C5.1, C6.1, D1.A, IC2A.G1, IC2P.VCC, IC3P.VCC, JP1.1, LED1.A, PCB1.5V0@1, PCB1.5V0@2, R2.2, U$1.OUT, U1.5V
- removed net RPI_RXD: JP1.3, PCB1.RXD0/GPIO15
- removed net RPI_TXD: JP1.2, PCB1.TXD0/GPIO14
- new net +12V: C1.+, C11.+, C12.1, C13.1, C14.1, C15.1, C16.1, C17.1, C9.1, IC2.IN, Q11.S, Q13.S, Q3.S, Q5.S, Q7.S, Q9.S, R11.2, R15.2, R19.2, R23.2, R28.2, R6.2, X1-1.KL
- new net DM: IC4.USBDM, X15G$1.2
- new net DP: IC4.USBDP, X15G$1.3
- new net D_ENABLE: SV5.4, U$1.PC9
- new net D_IM1: SV4.3, U$1.PF4
- new net D_IM2: SV4.4, U$1.PF5
- new net D_RESET: SV5.1, U$1.PC6
- new net D_RS: SV5.2, U$1.PC7
- new net D_RW: SV5.3, U$1.PC8
- new net ID: X15G$1.4
- new net N$1: JP1.1, JP2.2
- new net N$12: R3.1, R5.A, R5.S
- new net N$23: R30.1, R31.1, SV2.1, SV2.2, SV2.3
- new net N$24: U$1.PA11
- new net N$25: U$1.PA12
- new net N$27: R38.2, SJ1.2, X15S.S3
- new net N$32: C20.1, IC4.3V3OUT
- new net NRST: JP1.5, U$1.NRST
- new net OSC_IN: C6.1, Q1.1, U$1.PF0/OSC_IN
- new net OSC_OUT: C7.1, Q1.2, U$1.PF1/OSC_OUT
- new net PA10: U$1.PA10
- new net PA5: U$1.PA5
- new net SPI1_MISO: SV5.7, U$1.PB4
- new net SPI1_MOSI: SV5.6, U$1.PB5
- new net SPI1_SCK: SV5.5, U$1.PB3
- new net SW1: R32.2, S1.P, S1.P1
- new net SW2: R33.2, S2.P, S2.P1
- new net SW3: R34.2, S3.P, S3.P1
- new net SW4: R35.2, S4.P, S4.P1
- new net SWCLK: JP1.2, U$1.SWCLK/PA14
- new net SWDIO: JP1.4, U$1.SWDIO/PA13
- new net USART1_RX: IC4.TXD, JP3.2, U$1.PB7
- new net USART1_TX: IC4.RXD, JP3.3, U$1.PB6
- new net USART2_RX: SV1.8, U$1.PA3
- new net USART2_TX: SV1.1, U$1.PA2
- new net VBUS: C19.1, R37.1, X15G$1.1
- new net VCCUSB: C18.+, C2.1, IC4.VCC, IC4.VCCIO, R37.2
- new net WIFI_RESET: R36.2, SV1.4, SV1.6, U$1.PA1
- net +3V3: now also C10.1, C3.1, C4.1, C5.1, C8.1, IC1P.VCC, IC2.OUT, IC3A.G1, IC3P.VCC, JP2.1, LED1.A, R25.2, R30.2, R31.2, R7.2, S1.S, S1.S1, S2.S, S2.S1, S3.S, S3.S1, S4.S, S4.S1, SV1.2, SV4.2, U$1.VDDA, U$1.VDD_1, U$1.VDD_2; no longer R4.2, U1.3V
- net ERROR_LED: now also U$1.PC13
- net FREQ: now also IC1A.Y, U$1.PA9; no longer IC3A.Y
- net GND: now also C10.2, C11.-, C18.-, C19.2, C2.2, C20.2, C3.2, C7.2, C8.2, C9.2, D1.A, IC1P.GND, IC4.GND, IC4.GND@1, IC4.GND@2, IC4.GND@A, J10-3.S, J11-3.S, J12-3.S, J13-3.S, J14-3.S, J15-3.S, J16-3.S, J9-3.S, JP1.3, JP3.4, Q12.E, Q4.E, Q8.E, R1.1, R14.1, R22.1, R27.1, R3.2, R32.1, R33.1, R34.1, R35.1, R36.1, R38.1, R39.1, R4.1, SJ1.1, SV1.7, SV3.1, SV3.2, SV3.3, SV4.1, U$1.BOOT0, U$1.VSSA, U$1.VSS_1, U$1.VSS_2, X10-2.1, X11-2.1, X12-2.1, X13-2.1, X15G$1.5, X8-2.1, X9-2.1; no longer C3.-, D7.A, IC2P.GND, JP1.4, PCB1.GND@1, PCB1.GND@2, PCB1.GND@3, PCB1.GND@4, PCB1.GND@5, PCB1.GND@6, PCB1.GND@7, PCB1.GND@8, Q1.E, Q5.E, Q9.E, R1.2, R17.1, R25.1, R26.1, R29.1, R3.1, R9.1, U1.GND
- net N$10: now also Q6.C, R16.1; no longer Q9.C, R27.1
- net N$11: now also Q6.B, R13.2, R14.2; no longer Q9.B, R23.2, R25.2
- net N$13: now also C15.2, Q9.G, R19.1, R20.2; no longer C8.2, Q4.G, R12.2, R6.1
- net N$14: now also Q8.C, R20.1; no longer Q2.C, R12.1
- net N$15: now also Q8.B, R17.2, R18.2; no longer Q2.B, R10.2, R8.2
- net N$16: now also C16.2, Q11.G, R23.1, R24.2; no longer C10.2, Q8.G, R14.1, R20.2
- net N$17: now also Q10.C, R24.1; no longer Q6.C, R20.1
- net N$18: now also Q10.B, R21.2, R22.2; no longer Q6.B, R16.2, R18.2
- net N$19: now also C17.2, Q13.G, R28.1, R29.2; no longer C12.2, Q12.G, R22.1, R28.2
- net N$2: now also C13.2, Q5.G, R11.1, R12.2; no longer C9.2, Q7.G, R13.1, R19.2
- net N$20: now also IC2.ADJ, R5.E, R7.1; no longer R1.1, R2.1, U$1.ADJ
- net N$21: now also Q12.C, R29.1; no longer Q10.C, R28.1
- net N$22: now also Q12.B, R27.2; no longer Q10.B, R24.2
- net N$29: now also R39.2; no longer R29.2
- net N$3: now also C12.2, R6.1, R8.2; no longer C7.2, R11.2, R5.1
- net N$4: now also Q2.C, R8.1; no longer Q1.C, R11.1
- net N$5: now also Q2.B, R2.2, R4.2; no longer Q1.B, R7.2, R9.2
- net N$6: now also Q4.C, R12.1; no longer Q5.C, R19.1
- net N$7: now also Q4.B, R10.2, R9.2; no longer Q5.B, R15.2, R17.2
- net N$8: now also C14.2, Q7.G, R15.1, R16.2; no longer C11.2, Q11.G, R21.1, R27.2
- net N$9: now also R1.2; no longer R3.2
- net PA4: now also R2.1, U$1.PA4; no longer R7.1
- net PA6: now also R9.1, U$1.PA6; no longer R15.1
- net PA7: now also R13.1, U$1.PA7; no longer R23.1
- net PA8: now also R26.1, U$1.PA8; no longer R24.1
- net PB0: now also R17.1, U$1.PB0; no longer R8.1
- net PB10: now also R21.1, U$1.PB10; no longer R16.1
- net S1_3V: now also IC3A.Y0, J9-1.S; no longer IC2A.Y0
- net S1_DAT: now also IC1A.D0, J9-2.S; no longer IC3A.D0
- net S2_3V: now also IC3A.Y1, J10-1.S; no longer IC2A.Y1
- net S2_DAT: now also IC1A.D1, J10-2.S; no longer IC3A.D1
- net S3_3V: now also IC3A.Y2, J11-1.S; no longer IC2A.Y2
- net S3_DAT: now also IC1A.D2, J11-2.S; no longer IC3A.D2
- net S4_3V: now also IC3A.Y3, J12-1.S; no longer IC2A.Y3
- net S4_DAT: now also IC1A.D3, J12-2.S; no longer IC3A.D3
- net S5_3V: now also IC3A.Y4, J13-1.S; no longer IC2A.Y4
- net S5_DAT: now also IC1A.D4, J13-2.S; no longer IC3A.D4
- net S6_3V: now also IC3A.Y5, J14-1.S; no longer IC2A.Y5
- net S6_DAT: now also IC1A.D5, J14-2.S; no longer IC3A.D5
- net S7_3V: now also IC3A.Y6, J15-1.S; no longer IC2A.Y6
- net S7_DAT: now also IC1A.D6, J15-2.S; no longer IC3A.D6
- net S8_3V: now also IC3A.Y7, J16-1.S; no longer IC2A.Y7
- net S8_DAT: now also IC1A.D7, J16-2.S; no longer IC3A.D7
- net SEN_ENABLE: now also IC1A.G, IC3A.G2A, IC3A.G2B, R25.1, U$1.PB15; no longer IC2A.G2A, IC2A.G2B, IC3A.G, R4.1
- net SEN_SEL0: now also IC1A.A, U$1.PB14; no longer IC2A.A
- net SEN_SEL1: now also IC1A.B, U$1.PB13; no longer IC2A.B
- net SEN_SEL2: now also IC1A.C, U$1.PB12; no longer IC2A.C
- net WP1: now also D1.C, X8-1.1; no longer D2.C
- net WP2: now also D2.C, Q5.D, X9-1.1; no longer D4.C, Q7.D
- net WP3: now also D3.C, Q7.D, X10-1.1; no longer D6.C, Q11.D
- net WP4: now also D4.C, Q9.D, X11-1.1; no longer D3.C, Q4.D
- net WP5: now also Q11.D, X12-1.1; no longer Q8.D
- net WP6: now also D6.C, Q13.D, X13-1.1; no longer D7.C, Q12.D
Other:
- note added: "display:"
